File: Ski-Tracker-KiCad/Ski-Tracker.kicad_pcb (KiCad board)
At the start: 2 copper layers, 35 x 65.2 mm, 20 parts, among them J2 Conn_01x02_Pin, J3 Conn_01x05_Socket, SW1 SW_SPDT, U1 LSM6DSOXTR, U2 BMP388, U3 MCP73831T-2ACI/MC

Commit message: small changes
Parts:
- added D3: LED, LED_SMD:LED_0805_2012Metric, F.Cu at (133.8, 85.9)
- added D4: LED, LED_SMD:LED_0805_2012Metric, F.Cu at (133.7, 82.5)
- added D5: LED, LED_SMD:LED_0805_2012Metric, F.Cu at (133.8, 79.0)
- added R7: 220, Resistor_SMD:R_0603_1608Metric, F.Cu at (125.2, 94.5)
- added R8: 220, Resistor_SMD:R_0603_1608Metric, F.Cu at (125.2, 91.4)
- added R9: 220, Resistor_SMD:R_0603_1608Metric, F.Cu at (125.3, 87.9)
- C3: value 0.1uF -> 4.7uF; footprint Capacitor_SMD:C_0402_1005Metric -> Capacitor_SMD:C_0805_2012Metric
- C6: footprint Capacitor_SMD:C_0402_1005Metric -> Capacitor_SMD:C_0805_2012Metric
- moved C3 14.8 mm to (125.0, 66.4), turned to -90 degrees
- moved D2 2.00 mm to (133.8, 72.2)
- moved C2 1.08 mm to (129.8, 81.5)
- moved U1 0.98 mm to (129.6, 85.6)
- moved R4 0.06 mm to (131.8, 75.4)
Connections:
- A1 pad 24: unconnected-(A1-GPIO18-Pad24) -> /LED1
- A1 pad 25: unconnected-(A1-GPIO19-Pad25) -> /LED2
- A1 pad 26: unconnected-(A1-GPIO20-Pad26) -> /LED3
Routing:
- net GND: track 34.6 -> 3.90 mm, vias 26 -> 29
- net Net-(D5-A): track 0.00 -> 14.5 mm
- net Net-(D4-A): track 0.00 -> 12.2 mm
- net Net-(D3-A): track 0.00 -> 11.5 mm
- net /LED1: track 0.00 -> 4.41 mm
- net /LED2: track 0.00 -> 4.13 mm
- net /LED3: track 0.00 -> 3.88 mm
- net /STAT: track 2.14 -> 3.95 mm
- net /SDA: track 59.0 -> 57.2 mm
- net Net-(D2-A): track 1.47 -> 2.62 mm
- net /SCL: track 54.4 -> 53.5 mm
- net +3.3V: track 50.2 -> 49.3 mm
- net /VBUS: track 49.5 -> 50.0 mm

Commit message: changed diode value
Parts:
- D1: value 1N5817 -> MBR0520
Changed lines of the file:
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@@
 			)
 		)
-		(property "Value" "1N5817"
+		(property "Value" "MBR0520"
 			(at 0 4 0)
 			(layer "F.Fab")

Commit message: Status LED
Parts:
- moved J2 2.45 mm to (133.4, 54.2), turned to 90 degrees
Connections:
- net +3.3V renamed +3V3
Routing:
- net /VBAT: track 33.3 -> 31.1 mm

Commit message: KiCad 10 update
Parts:
- moved C6 16.0 mm to (125.2, 71.3), turned to -90 degrees
- moved C1 4.36 mm to (130.2, 83.1)
- moved C2 1.10 mm to (130.2, 80.5)
- moved C4 0.96 mm to (129.5, 78.0), turned to 180 degrees
Routing:
- net /VBAT: track 31.1 -> 29.5 mm
- net /ADC2: track 10.4 -> 11.5 mm
- net +3V3: track 49.3 -> 48.5 mm
- net GND: vias 29 -> 28
